Commit message: Began to fix camera for better oracle

File: docker_volume/environments/assets/robot/ur10e.urdf (robot description, URDF)
Before this commit: robot ur10e, 26 links, 25 joints
Links:
- link realsense_mount_base_link: geometry visual mesh filename=../meshes/realsense_mount.stl scale=0.0001 0.0001 0.0001
- link tcp_link: geometry visual sphere radius=0.025
